Commit message: 添加debug测试

File: robots/BQR3W_350_fix/urdf/BQR3W_350.urdf (robot description, URDF)
Before this commit: robot quadruped_new, 21 links, 20 joints
Links:
- link Wheel1Link: geometry collision cylinder length=0.01 radius=0.125; visual box size=0.02 0.01 0.05
- link Wheel2Link: geometry collision cylinder length=0.01 radius=0.125; visual box size=0.02 0.01 0.05
- link Wheel3Link: geometry collision cylinder length=0.01 radius=0.125; visual box size=0.02 0.01 0.05
- link Wheel4Link: geometry collision cylinder length=0.01 radius=0.125; visual box size=0.02 0.01 0.05
